Commit message: stuff

File: description/robot.urdf.xacro (robot description, xacro)
@@ -12,4 +12,5 @@
     <xacro:include filename="lidar.xacro" />
     <xacro:include filename="camera.xacro" />
+    <!-- <xacro:include filename="xarm_xacros/xarm.xacro" /> -->
     <!-- <xacro:include filename="xarm.urdf"/> -->
     <!-- <xacro:include filename="depth_camera.xacro" /> -->

File: description/xarm_xacros/xarm_v2.urdf (robot description, URDF)
Before this commit: robot xarm, 5 links, 6 joints
Links:
- link xarm_3_link: geometry collision mesh filename=file://$(find xarm_description)/meshes/stls/link3.stl scale=1.0 1.0 1.0; visual mesh filename=file://$(find xarm_description)/meshes/stls/link3.stl scale=1.0 1.0 1.0
- link xarm_4_link: geometry collision mesh filename=file://$(find xarm_description)/meshes/stls/link4.stl scale=1.0 1.0 1.0; visual mesh filename=file://$(find xarm_description)/meshes/stls/link4.stl scale=1.0 1.0 1.0
- link xarm_5_link: geometry collision mesh filename=file://$(find xarm_description)/meshes/stls/link5.stl scale=1.0 1.0 1.0; visual mesh filename=file://$(find xarm_description)/meshes/stls/link5.stl scale=1.0 1.0 1.0
- link xarm_6_link: geometry collision mesh filename=file://$(find xarm_description)/meshes/stls/link6.stl scale=1.0 1.0 1.0; visual mesh filename=file://$(find xarm_description)/meshes/stls/link6.stl scale=1.0 1.0 1.0
- link xarm_base_link: mass None -> 1; geometry collision mesh filename=file://$(find xarm_description)/meshes/stls/base.stl scale=1.0 1.0 1.0; visual mesh filename=file://$(find xarm_description)/meshes/stls/base.stl scale=1.0 1.0 1.0
Joints:
- removed joint xarm_joint

Commit message: got robot arm working

File: description/robot.urdf.xacro (robot description, xacro)
@@ -12,5 +12,6 @@
     <xacro:include filename="lidar.xacro" />
     <xacro:include filename="camera.xacro" />
-    <!-- <xacro:include filename="xarm_xacros/xarm.xacro" /> -->
+    <xacro:include filename="xarm_xacros/xarm.xacro" />
+    <xacro:include filename="xarm_xacros/ros2_control_params.xacro" />
     <!-- <xacro:include filename="xarm.urdf"/> -->
     <!-- <xacro:include filename="depth_camera.xacro" /> -->

File: description/ros2_control.xacro (robot description, xacro)
@@ -93,11 +93,11 @@
         </ros2_control>
     </xacro:if>
+     <!-- <plugin name="gz_ros2_control::GazeboSimROS2ControlPlugin" filename="libgz_ros2_control-system.so"> -->
     <!-- Gazebo ROS2 control plugin -->
-    <gazebo>
+    <!-- <gazebo>
         <plugin filename="gz_ros2_control-system" name="gz_ros2_control::GazeboSimROS2ControlPlugin">
-        <!-- <plugin name="gz_ros2_control::GazeboSimROS2ControlPlugin" filename="libgz_ros2_control-system.so"> -->
             <parameters>$(find articubot_one)/config/my_controllers.yaml</parameters>
             <parameters>$(find articubot_one)/config/gaz_ros2_ctl_use_sim.yaml</parameters>
         </plugin>
-    </gazebo>
+    </gazebo> -->
 </robot>

File: description/xarm_xacros/ros2_control.arm.xacro (robot description, xacro)
@@ -105,5 +105,6 @@
   </xacro:unless>
   <xacro:if value="$(arg sim_mode)">
-    <ros2_control name="GazeboSystem" type="system">
+    <!-- <ros2_control name="GazeboSystem" type="system"> -->
+    <ros2_control name="arm_system" type="system">
         <hardware>
             <plugin>gz_ros2_control/GazeboSimSystem</plugin>
@@ -216,10 +217,10 @@
     </ros2_control>
   </xacro:if>
-  <gazebo>
+  <!-- <plugin name="gz_ros2_control::GazeboSimROS2ControlPlugin" filename="libgz_ros2_control-system.so"> -->
+  <!-- <gazebo>
       <plugin filename="gz_ros2_control-system" name="gz_ros2_control::GazeboSimROS2ControlPlugin">
-      <!-- <plugin name="gz_ros2_control::GazeboSimROS2ControlPlugin" filename="libgz_ros2_control-system.so"> -->
           <parameters>$(find articubot_one)/config/xarm_controllers.yaml</parameters>
           <parameters>$(find articubot_one)/config/gaz_ros2_ctl_use_sim.yaml</parameters>
       </plugin>
-  </gazebo>
+  </gazebo> -->
 </robot>

File: description/xarm_xacros/xarm.xacro (robot description, xacro)
@@ -1,7 +1,11 @@
 <?xml version="1.0"?>
 <robot xmlns:xacro="http://ros.org/wiki/xacro" name="xarm">
+    <xacro:property name="chassis_length1" value="0.432"/>
+    <xacro:property name="chassis_width1" value="0.432"/>
+    <xacro:property name="chassis_height1" value="0.048"/>
     <!-- <xacro:property name="eef" value="eef_3_finger"/> -->
     <xacro:property name="eef" value="eef_2_finger"/>
     <xacro:arg name="sim_mode" default="true"/>
+    <!-- <xacro:include filename="$(find articubot_one)/description/robot_dimensions.xacro"/> -->
     <!-- <xacro:include filename="$(find xarm_description)/urdf/xarm.urdf"/> -->
     <xacro:include filename="xarm_v2.urdf"/>
@@ -9,5 +13,5 @@
         <parent link="chassis"/>
         <child link="xarm_base_link"/>
-        <origin xyz="0.0 0.0 0.0" rpy="0.0 0.0 0.0"/>
+        <origin xyz="${chassis_length1/4+0.02} ${chassis_width1/4+0.02} ${chassis_height1}" rpy="0.0 0.0 -${pi/2}"/>
     </joint>
     <xacro:include filename="ros2_control.arm.xacro" />
